Commit message: genesis sim and now walks

File: sim/resources/stompymicro/robot.urdf (robot description, URDF)
Before this commit: robot opus, 18 links, 17 joints
Links:
- removed link left_knee_pitch_motor
- removed link right_knee_pitch_motor
- added link ankle_pitch_left, mass 0.164074011; collision mesh filename=meshes/ankle_pitch_left.stl; visual mesh filename=meshes/ankle_pitch_left.stl
- added link ankle_pitch_right, mass 0.164074011; collision mesh filename=meshes/ankle_pitch_right.stl; visual mesh filename=meshes/ankle_pitch_right.stl
- link knee_pitch_left: mass 0.017415556 -> 0.017415406
- link knee_pitch_right: mass 0.017415406 -> 0.017415556
Joints:
- joint left_ankle_pitch: origin xyz=0.0 -0.07771999985844844 -0.000499991045895997 rpy=9.282041357749903e-08 0.0 0.0 -> xyz=0.0 0.06 0 rpy=9.282041357749903e-08 0.0 0.0; parent left_knee_pitch_motor -> ankle_pitch_left
- joint left_elbow_yaw: limit lower=-1.5707963 upper=1.5707963 effort=80 velocity=5 -> lower=1.5707963 upper=4.71 effort=80 velocity=5
- joint left_hip_pitch: origin xyz=0.045549819648300315 -0.0003268960191209584 -0.10384882247403085 rpy=1.5707963535897942 -4.6410206566704915e-08 1.5707963000000003 -> xyz=0.045549819648300315 -0.0003268960191209584 -0.09684882247403085 rpy=1.5707963535897942 -4.6410206566704915e-08 1.5707963000000003
- joint left_hip_roll: child knee_pitch_right -> knee_pitch_left; origin xyz=0.0 0.06776001212246713 0.014999999060838654 rpy=-1.5707963071795865 0.0 0.0 -> xyz=0.0 0.07776001212246713 0.014999999060838654 rpy=-1.5707963071795865 0.0 0.0
- joint left_hip_yaw: limit lower=-1.5707963 upper=0.087266463 effort=80 velocity=5 -> lower=-0.1 upper=0.3 effort=80 velocity=5; origin xyz=-0.02550000297464769 -0.012500001 0.01936000008172467 rpy=-3.1415926071795863 -1.5707963 0.0 -> xyz=-0.02550000297464769 0 0.01936000008172467 rpy=-3.1415926071795863 -1.5707963 0.0
- joint left_knee_pitch: child left_knee_pitch_motor -> ankle_pitch_left; origin xyz=-0.018825 0 0.02221 rpy=-1.5707963 0 -1.5707963 -> xyz=0.020825 0 0.03271 rpy=1.5707963 0 -1.5707963; parent knee_pitch_right -> knee_pitch_left
- joint righ_elbow_yaw: limit lower=-1.5707963 upper=1.5707963 effort=80 velocity=5 -> lower=1.5707963 upper=4.71 effort=80 velocity=5
- joint right_ankle_pitch: origin xyz=0.0 0.07772000162667812 2.0870670330852548e-09 rpy=9.282041357749903e-08 0.0 0.0 -> xyz=0.0 -0.06 0 rpy=9.282041357749903e-08 0.0 0.0; parent right_knee_pitch_motor -> ankle_pitch_right
- joint right_hip_pitch: origin xyz=-0.045750183202404315 -0.00032689585567163837 -0.10384882247403085 rpy=-1.570796353589792 -4.6410206566704915e-08 1.5707963000000003 -> xyz=-0.045750183202404315 -0.00032689585567163837 -0.09684882247403085 rpy=-1.570796353589792 -4.6410206566704915e-08 1.5707963000000003
- joint right_hip_roll: child knee_pitch_left -> knee_pitch_right; origin xyz=0.0 0.06776001387753285 0.015000000939161373 rpy=-1.5707963 0.0 0.0 -> xyz=0.0 0.07776001212246713 0.015000000939161373 rpy=-1.5707963 0.0 0.0
- joint right_hip_yaw: limit lower=-0.087266463 upper=1.5707963 effort=80 velocity=5 -> lower=-0.3 upper=0.1 effort=80 velocity=5; origin xyz=-0.02550000162875169 0.012500001141551514 0.019359999918275368 rpy=9.282041333256968e-08 1.5707963000000005 0.0 -> xyz=-0.02550000162875169 0 0.019359999918275368 rpy=9.282041333256968e-08 1.5707963000000005 0.0
- joint right_knee_pitch: child right_knee_pitch_motor -> ankle_pitch_right; origin xyz=0.018825 0 0.02221 rpy=1.5707963 0 -1.5707963 -> xyz=-0.020825 0 0.03271 rpy=-1.5707963 0 -1.5707963; parent knee_pitch_left -> knee_pitch_right

File: sim/resources/stompymicro/robot_fixed.urdf (robot description, URDF)
Before this commit: robot opus, 18 links, 17 joints
Links:
- removed link left_knee_pitch_motor
- removed link right_knee_pitch_motor
- added link ankle_pitch_left, mass 0.164074011; collision mesh filename=meshes/ankle_pitch_left.stl; visual mesh filename=meshes/ankle_pitch_left.stl
- added link ankle_pitch_right, mass 0.164074011; collision mesh filename=meshes/ankle_pitch_right.stl; visual mesh filename=meshes/ankle_pitch_right.stl
- link Torso: mass 1.4248854441999999 -> 1.8248854441999999
- link knee_pitch_left: mass 0.017415556 -> 0.017415406
- link knee_pitch_right: mass 0.017415406 -> 0.017415556
Joints:
- removed joint righ_elbow_yaw
- added joint right_elbow_yaw: type revolute, parent right_shoulder_yaw_motor, child right_hand, origin xyz=-0.030003116165437632 -0.06434189265302206 -0.00015000392836930906 rpy=3.141592518707449 -1.961380480253183e-08 2.7052603000000013, axis 0 0 1, limit lower=1.5707963 upper=4.71 effort=2 velocity=10
- joint left_ankle_pitch: limit lower=-1.0471976 upper=1.0471976 effort=2 velocity=10 -> lower=-1.5707963 upper=1.5707963 effort=2 velocity=10; origin xyz=0.0 -0.07771999985844844 -0.000499991045895997 rpy=9.282041357749903e-08 0.0 0.0 -> xyz=0.0 0.06 0 rpy=9.282041357749903e-08 0.0 0.0; parent left_knee_pitch_motor -> ankle_pitch_left
- joint left_elbow_yaw: limit lower=-1.5707963 upper=1.5707963 effort=80 velocity=5 -> lower=1.5707963 upper=4.71 effort=2 velocity=10; type fixed -> revolute
- joint left_hip_pitch: origin xyz=0.045549819648300315 -0.0003268960191209584 -0.10384882247403085 rpy=1.5707963535897942 -4.6410206566704915e-08 1.5707963000000003 -> xyz=0.045549819648300315 -0.0003268960191209584 -0.09684882247403085 rpy=1.5707963535897942 -4.6410206566704915e-08 1.5707963000000003
- joint left_hip_roll: child knee_pitch_right -> knee_pitch_left; origin xyz=0.0 0.06776001212246713 0.014999999060838654 rpy=-1.5707963071795865 0.0 0.0 -> xyz=0.0 0.07776001212246713 0.014999999060838654 rpy=-1.5707963071795865 0.0 0.0
- joint left_hip_yaw: limit lower=-1.5707963 upper=0.087266463 effort=2 velocity=10 -> lower=-0.1 upper=0.3 effort=2 velocity=10; origin xyz=-0.02550000297464769 -0.012500001 0.01936000008172467 rpy=-3.1415926071795863 -1.5707963 0.0 -> xyz=-0.02550000297464769 0 0.01936000008172467 rpy=-3.1415926071795863 -1.5707963 0.0
- joint left_knee_pitch: child left_knee_pitch_motor -> ankle_pitch_left; limit lower=-1.0471976 upper=0 effort=2 velocity=10 -> lower=-1.5707963 upper=1.5707963 effort=2 velocity=10; origin xyz=-0.018825 0 0.02221 rpy=-1.5707963 0 -1.5707963 -> xyz=0.020825 0 0.03271 rpy=1.5707963 0 -1.5707963; parent knee_pitch_right -> knee_pitch_left
- joint right_ankle_pitch: limit lower=-1.0471976 upper=1.0471976 effort=2 velocity=10 -> lower=-1.5707963 upper=1.5707963 effort=2 velocity=10; origin xyz=0.0 0.07772000162667812 2.0870670330852548e-09 rpy=9.282041357749903e-08 0.0 0.0 -> xyz=0.0 -0.06 0 rpy=9.282041357749903e-08 0.0 0.0; parent right_knee_pitch_motor -> ankle_pitch_right
- joint right_hip_pitch: origin xyz=-0.045750183202404315 -0.00032689585567163837 -0.10384882247403085 rpy=-1.570796353589792 -4.6410206566704915e-08 1.5707963000000003 -> xyz=-0.045750183202404315 -0.00032689585567163837 -0.09684882247403085 rpy=-1.570796353589792 -4.6410206566704915e-08 1.5707963000000003
- joint right_hip_roll: child knee_pitch_left -> knee_pitch_right; origin xyz=0.0 0.06776001387753285 0.015000000939161373 rpy=-1.5707963 0.0 0.0 -> xyz=0.0 0.07776001212246713 0.015000000939161373 rpy=-1.5707963 0.0 0.0
- joint right_hip_yaw: limit lower=-0.087266463 upper=1.5707963 effort=2 velocity=10 -> lower=-0.3 upper=0.1 effort=2 velocity=10; origin xyz=-0.02550000162875169 0.012500001141551514 0.019359999918275368 rpy=9.282041333256968e-08 1.5707963000000005 0.0 -> xyz=-0.02550000162875169 0 0.019359999918275368 rpy=9.282041333256968e-08 1.5707963000000005 0.0
- joint right_knee_pitch: child right_knee_pitch_motor -> ankle_pitch_right; limit lower=0 upper=1.0471976 effort=2 velocity=10 -> lower=-1.5707963 upper=1.5707963 effort=2 velocity=10; origin xyz=0.018825 0 0.02221 rpy=1.5707963 0 -1.5707963 -> xyz=-0.020825 0 0.03271 rpy=-1.5707963 0 -1.5707963; parent knee_pitch_left -> knee_pitch_right

Commit message: genesis sim

File: sim/resources/stompymicro/robot.urdf (robot description, URDF)
Before this commit: robot opus, 18 links, 17 joints
Links:
- removed link left_knee_pitch_motor
- removed link right_knee_pitch_motor
- added link ankle_pitch_left, mass 0.164074011; collision mesh filename=meshes/ankle_pitch_left.stl; visual mesh filename=meshes/ankle_pitch_left.stl
- added link ankle_pitch_right, mass 0.164074011; collision mesh filename=meshes/ankle_pitch_right.stl; visual mesh filename=meshes/ankle_pitch_right.stl
- link knee_pitch_left: mass 0.017415556 -> 0.017415406
- link knee_pitch_right: mass 0.017415406 -> 0.017415556
Joints:
- joint left_ankle_pitch: parent left_knee_pitch_motor -> ankle_pitch_left
- joint left_elbow_yaw: limit lower=-1.5707963 upper=1.5707963 effort=80 velocity=5 -> lower=1.5707963 upper=4.71 effort=80 velocity=5
- joint left_hip_roll: child knee_pitch_right -> knee_pitch_left
- joint left_knee_pitch: child left_knee_pitch_motor -> ankle_pitch_left; origin xyz=-0.018825 0 0.02221 rpy=-1.5707963 0 -1.5707963 -> xyz=0.018825 0 0.02221 rpy=1.5707963 0 -1.5707963; parent knee_pitch_right -> knee_pitch_left
- joint righ_elbow_yaw: limit lower=-1.5707963 upper=1.5707963 effort=80 velocity=5 -> lower=1.5707963 upper=4.71 effort=80 velocity=5
- joint right_ankle_pitch: origin xyz=0.0 0.07772000162667812 2.0870670330852548e-09 rpy=9.282041357749903e-08 0.0 0.0 -> xyz=0.0 0 0 rpy=9.282041357749903e-08 0.0 0.0; parent right_knee_pitch_motor -> ankle_pitch_right
- joint right_hip_roll: child knee_pitch_left -> knee_pitch_right
- joint right_knee_pitch: child right_knee_pitch_motor -> ankle_pitch_right; origin xyz=0.018825 0 0.02221 rpy=1.5707963 0 -1.5707963 -> xyz=-0.018825 0 0.02221 rpy=-1.5707963 0 -1.5707963; parent knee_pitch_left -> knee_pitch_right

Commit message: fixed train

File: sim/resources/stompymicro/robot.urdf (robot description, URDF)
Before this commit: robot opus, 18 links, 17 joints
Joints:
- joint left_ankle_pitch: origin xyz=0.0 -0.07771999985844844 -0.000499991045895997 rpy=9.282041357749903e-08 0.0 0.0 -> xyz=0.0 0.06 0 rpy=9.282041357749903e-08 0.0 0.0
- joint left_hip_pitch: origin xyz=0.045549819648300315 -0.0003268960191209584 -0.10384882247403085 rpy=1.5707963535897942 -4.6410206566704915e-08 1.5707963000000003 -> xyz=0.045549819648300315 -0.0003268960191209584 -0.09684882247403085 rpy=1.5707963535897942 -4.6410206566704915e-08 1.5707963000000003
- joint left_hip_roll: origin xyz=0.0 0.06776001212246713 0.014999999060838654 rpy=-1.5707963071795865 0.0 0.0 -> xyz=0.0 0.07776001212246713 0.014999999060838654 rpy=-1.5707963071795865 0.0 0.0
- joint left_hip_yaw: limit lower=-1.5707963 upper=0.087266463 effort=80 velocity=5 -> lower=-0.1 upper=0.3 effort=80 velocity=5; origin xyz=-0.02550000297464769 -0.012500001 0.01936000008172467 rpy=-3.1415926071795863 -1.5707963 0.0 -> xyz=-0.02550000297464769 0 0.01936000008172467 rpy=-3.1415926071795863 -1.5707963 0.0
- joint left_knee_pitch: origin xyz=0.018825 0 0.02221 rpy=1.5707963 0 -1.5707963 -> xyz=0.020825 0 0.03271 rpy=1.5707963 0 -1.5707963
- joint right_ankle_pitch: origin xyz=0.0 0 0 rpy=9.282041357749903e-08 0.0 0.0 -> xyz=0.0 -0.06 0 rpy=9.282041357749903e-08 0.0 0.0
- joint right_hip_pitch: origin xyz=-0.045750183202404315 -0.00032689585567163837 -0.10384882247403085 rpy=-1.570796353589792 -4.6410206566704915e-08 1.5707963000000003 -> xyz=-0.045750183202404315 -0.00032689585567163837 -0.09684882247403085 rpy=-1.570796353589792 -4.6410206566704915e-08 1.5707963000000003
- joint right_hip_roll: origin xyz=0.0 0.06776001387753285 0.015000000939161373 rpy=-1.5707963 0.0 0.0 -> xyz=0.0 0.07776001212246713 0.015000000939161373 rpy=-1.5707963 0.0 0.0
- joint right_hip_yaw: limit lower=-0.087266463 upper=1.5707963 effort=80 velocity=5 -> lower=-0.3 upper=0.1 effort=80 velocity=5; origin xyz=-0.02550000162875169 0.012500001141551514 0.019359999918275368 rpy=9.282041333256968e-08 1.5707963000000005 0.0 -> xyz=-0.02550000162875169 0 0.019359999918275368 rpy=9.282041333256968e-08 1.5707963000000005 0.0
- joint right_knee_pitch: origin xyz=-0.018825 0 0.02221 rpy=-1.5707963 0 -1.5707963 -> xyz=-0.020825 0 0.03271 rpy=-1.5707963 0 -1.5707963

File: sim/resources/stompymicro/robot_fixed.urdf (robot description, URDF)
Before this commit: robot opus, 18 links, 17 joints
Links:
- removed link left_knee_pitch_motor
- removed link right_knee_pitch_motor
- added link ankle_pitch_left, mass 0.164074011; collision mesh filename=meshes/ankle_pitch_left.stl; visual mesh filename=meshes/ankle_pitch_left.stl
- added link ankle_pitch_right, mass 0.164074011; collision mesh filename=meshes/ankle_pitch_right.stl; visual mesh filename=meshes/ankle_pitch_right.stl
- link Torso: mass 1.4248854441999999 -> 1.8248854441999999
- link knee_pitch_left: mass 0.017415556 -> 0.017415406
- link knee_pitch_right: mass 0.017415406 -> 0.017415556
Joints:
- joint left_ankle_pitch: limit lower=-1.0471976 upper=1.0471976 effort=2 velocity=10 -> lower=-1.5707963 upper=1.5707963 effort=2 velocity=10; origin xyz=0.0 -0.07771999985844844 -0.000499991045895997 rpy=9.282041357749903e-08 0.0 0.0 -> xyz=0.0 0.06 0 rpy=9.282041357749903e-08 0.0 0.0; parent left_knee_pitch_motor -> ankle_pitch_left
- joint left_elbow_yaw: limit lower=-1.5707963 upper=1.5707963 effort=80 velocity=5 -> lower=1.5707963 upper=4.71 effort=80 velocity=5
- joint left_hip_pitch: origin xyz=0.045549819648300315 -0.0003268960191209584 -0.10384882247403085 rpy=1.5707963535897942 -4.6410206566704915e-08 1.5707963000000003 -> xyz=0.045549819648300315 -0.0003268960191209584 -0.09684882247403085 rpy=1.5707963535897942 -4.6410206566704915e-08 1.5707963000000003
- joint left_hip_roll: child knee_pitch_right -> knee_pitch_left; origin xyz=0.0 0.06776001212246713 0.014999999060838654 rpy=-1.5707963071795865 0.0 0.0 -> xyz=0.0 0.07776001212246713 0.014999999060838654 rpy=-1.5707963071795865 0.0 0.0
- joint left_hip_yaw: limit lower=-1.5707963 upper=0.087266463 effort=2 velocity=10 -> lower=-0.1 upper=0.3 effort=2 velocity=10; origin xyz=-0.02550000297464769 -0.012500001 0.01936000008172467 rpy=-3.1415926071795863 -1.5707963 0.0 -> xyz=-0.02550000297464769 0 0.01936000008172467 rpy=-3.1415926071795863 -1.5707963 0.0
- joint left_knee_pitch: child left_knee_pitch_motor -> ankle_pitch_left; limit lower=-1.0471976 upper=0 effort=2 velocity=10 -> lower=-1.5707963 upper=1.5707963 effort=2 velocity=10; origin xyz=-0.018825 0 0.02221 rpy=-1.5707963 0 -1.5707963 -> xyz=0.020825 0 0.03271 rpy=1.5707963 0 -1.5707963; parent knee_pitch_right -> knee_pitch_left
- joint righ_elbow_yaw: limit lower=-1.5707963 upper=1.5707963 effort=80 velocity=5 -> lower=1.5707963 upper=4.71 effort=80 velocity=5
- joint right_ankle_pitch: limit lower=-1.0471976 upper=1.0471976 effort=2 velocity=10 -> lower=-1.5707963 upper=1.5707963 effort=2 velocity=10; origin xyz=0.0 0.07772000162667812 2.0870670330852548e-09 rpy=9.282041357749903e-08 0.0 0.0 -> xyz=0.0 -0.06 0 rpy=9.282041357749903e-08 0.0 0.0; parent right_knee_pitch_motor -> ankle_pitch_right
- joint right_hip_pitch: origin xyz=-0.045750183202404315 -0.00032689585567163837 -0.10384882247403085 rpy=-1.570796353589792 -4.6410206566704915e-08 1.5707963000000003 -> xyz=-0.045750183202404315 -0.00032689585567163837 -0.09684882247403085 rpy=-1.570796353589792 -4.6410206566704915e-08 1.5707963000000003
- joint right_hip_roll: child knee_pitch_left -> knee_pitch_right; origin xyz=0.0 0.06776001387753285 0.015000000939161373 rpy=-1.5707963 0.0 0.0 -> xyz=0.0 0.07776001212246713 0.015000000939161373 rpy=-1.5707963 0.0 0.0
- joint right_hip_yaw: limit lower=-0.087266463 upper=1.5707963 effort=2 velocity=10 -> lower=-0.3 upper=0.1 effort=2 velocity=10; origin xyz=-0.02550000162875169 0.012500001141551514 0.019359999918275368 rpy=9.282041333256968e-08 1.5707963000000005 0.0 -> xyz=-0.02550000162875169 0 0.019359999918275368 rpy=9.282041333256968e-08 1.5707963000000005 0.0
- joint right_knee_pitch: child right_knee_pitch_motor -> ankle_pitch_right; limit lower=0 upper=1.0471976 effort=2 velocity=10 -> lower=-1.5707963 upper=1.5707963 effort=2 velocity=10; origin xyz=0.018825 0 0.02221 rpy=1.5707963 0 -1.5707963 -> xyz=-0.020825 0 0.03271 rpy=-1.5707963 0 -1.5707963; parent knee_pitch_left -> knee_pitch_right
